Commit message: Phase 1 complete: autonomous SLAM + Nav2 navigation
Adds the active-SLAM stack (slam_toolbox + Nav2 + explore_lite) and the
saved-map navigation flow. Covers all of Phase 1 from MISSION.md:
holonomic LeKiwi maps a room with the LD06 LiDAR via frontier exploration,
then drives autonomously to clicked goals on the saved map.

Key Nav2 config tuning for omni-drive (in nav2_params.yaml):
  - motion_model "Omni" for MPPI controller
  - min_y_velocity_threshold 0.001 (was 0.5 — diff-drive default that
    silently zeroed out lateral motion)
  - velocity_smoother Y components ±0.4 (was 0)
  - PreferForwardCritic disabled
  - inflation_radius 0.25 (sized for 1.6 m hallway in small_house)
  - amcl.set_initial_pose so global_costmap can activate without first
    needing a manual "2D Pose Estimate" click

Sim URDF (lekiwi.sim.urdf.xacro) skips the pantilt module because its
camera mount sits 5 cm above the LD06 plane and would otherwise show as
a permanent obstacle in front of the robot. Description package URDF
unchanged for real-robot use.

Adds MISSION.md (broader project goals) and rewrites README.md with the
multi-terminal reproduction recipe, since the all-in-one active_slam
launch has known DDS startup races on slow VMs.

Removes the custom auto_map.py — using explore_lite (battle-tested)
instead. m-explore-ros2 added to .gitignore (cloned separately on each
machine, has its own upstream .git).

Co-Authored-By: Claude Opus 4.7 (1M context) <noreply@anthropic.com>

File: src/lekiwi_gazebo/urdf/lekiwi.sim.urdf.xacro (robot description, xacro)
@@ -10,5 +10,11 @@
   <xacro:include filename="$(find lekiwi_description)/urdf/lekiwi.common.xacro"/>
   <xacro:include filename="$(find lekiwi_description)/urdf/base/base.module.xacro"/>
-  <xacro:include filename="$(find lekiwi_description)/urdf/pantilt/pantilt.module.xacro"/>
+  <!-- pantilt module is intentionally excluded in sim:
+       its tilt/camera mount sits 5 cm above the LD06 laser plane (0.16 m),
+       so forward beams hit the mount every scan and slam maps it as a wall
+       right in front of the robot — frontiers then cluster at the robot's
+       footprint and explore_lite can't pick a useful goal.
+       Re-enable for real-robot work where the camera matters. -->
+  <!-- <xacro:include filename="$(find lekiwi_description)/urdf/pantilt/pantilt.module.xacro"/> -->
   <xacro:include filename="$(find lekiwi_gazebo)/urdf/lekiwi.gazebo.xacro"/>
   <!-- Wheel geometry shared with the real-robot control xacro -->
@@ -31,7 +37,5 @@
     <origin xyz="0 0 ${wheel_radius - wheel_base_offset_z}" rpy="0 0 0"/>
   </xacro:lekiwi_base_module>
-  <xacro:pantilt_module parent="base_link">
-    <origin xyz="${pantilt_base_offset_x} 0 ${pantilt_base_offset_z}" rpy="0 0 0"/>
-  </xacro:pantilt_module>
+  <!-- pantilt skipped in sim — see comment in include block above -->
   <xacro:lekiwi_gazebo/>
 </robot>
