Commit message: Phase 2 v1: color-aware "go to the X ball" demo
Adds a sim camera, three colored balls in the world, a YOLOv8 detection
launch, and a goal-sender node that turns "/target_color: red|yellow|blue"
into a Nav2 NavigateToPose goal in front of the matching ball.

Sim URDF (lekiwi.gazebo.xacro):
  - New sim_camera_link / sim_camera_optical_frame, mounted at the real-robot
    height (~6.6 cm above floor) with proper ROS optical-convention rotation.
  - Gazebo camera sensor at 320x240 / 60° HFOV / 15 Hz publishing /camera/image
    and /camera/camera_info, bridged via ros_gz_bridge.yaml.
  - Description's existing camera_link is left untouched (its rotation is for
    the webcam visual mesh, not for sensor mounting).

World (small_house.sdf):
  - Three 10 cm radius "sports balls": yellow at (-2.5, 1.0), red at (-2.5, -1.0),
    blue at (-1.0, -2.0). All static so they don't roll. All recognized by
    YOLOv8 as COCO class "sports ball".

YOLO launch (yolo.launch.py):
  - Wraps yolo_bringup/yolo.launch.py with sensible CPU defaults: yolov8n.pt,
    192x192 inference, threshold 0.25, device=cpu. yolo_ros itself is a
    separate upstream clone (gitignored), as is the auto-downloaded model.

Goal-sender node (go_to_color_ball.py):
  - Subscribes to /target_color (std_msgs/String) + /yolo/detections +
    /camera/image + /camera/camera_info, publishes /goal_pose.
  - Color filter: samples bbox-center patch in HSV; matches red/yellow/blue
    by hue + saturation gate.
  - 2D→3D: projects bbox bottom-center to ground plane via camera intrinsics +
    map ← optical TF, then computes a goal stop_distance metres in front of
    the ball with yaw facing it.
  - Search loop: while target_color is set but no matching detection visible,
    spins 60° in place every 5 s; after a full ~360°, drives to the next
    waypoint (living room, hallway, bedroom, kitchen) and spins again.
  - Navigation lock: once a navigate-to-ball goal is published, suppresses
    the search timer until the robot arrives or 60 s timeout — prevents
    mid-trip diversions when the ball briefly drops out of frame.
  - Fine-adjust on arrival: P-controller-style yaw correction from bbox
    pixel error to centre the ball in the camera view; stops on
    convergence (±25 px), max 4 attempts, or 6 s without detection
    (means YOLO can't classify a ball that fills most of the frame =
    we're right in front of it, which is the desired end state).

Trigger from CLI:
  ros2 topic pub --once /target_color std_msgs/String "{data: red}"

Also drops the unused 22 MB lekiwi_base_old.stl that lingered after the
.gitignore change.

Co-Authored-By: Claude Opus 4.7 (1M context) <noreply@anthropic.com>

File: src/lekiwi_gazebo/urdf/lekiwi.gazebo.xacro (robot description, xacro)
@@ -26,4 +26,59 @@
         <dimensions>3</dimensions>
       </plugin>
+    </gazebo>
+    <!-- Forward-facing RGB camera, sim-only.
+         The description's camera_link rotates the visual mesh so its X axis
+         points DOWN (intentional for the webcam STL alignment) — that's the
+         wrong orientation for a Gazebo camera sensor (which expects link X
+         to point along the optical axis). Rather than fight that, we mount
+         a fresh sim-only sensor frame here with proper orientation, and
+         leave the description's camera/camera_link untouched.
+         Geometry matches the real robot: 11.4 cm forward of base_link,
+         2.6 cm up (≈6.6 cm above floor). Wheels and floor will appear in
+         the lower portion of the frame — that matches the physical setup. -->
+    <link name="sim_camera_link"/>
+    <joint name="sim_camera_joint" type="fixed">
+      <parent link="base_link"/>
+      <child link="sim_camera_link"/>
+      <origin xyz="0.114 0 0.022" rpy="0 0 0"/>
+    </joint>
+    <!-- Optical-convention frame: X right, Y down, Z forward (vs URDF body
+         frame which is X forward, Y left, Z up). Standard rpy that takes
+         body → optical is (-π/2, 0, -π/2). -->
+    <link name="sim_camera_optical_frame"/>
+    <joint name="sim_camera_optical_joint" type="fixed">
+      <parent link="sim_camera_link"/>
+      <child link="sim_camera_optical_frame"/>
+      <origin xyz="0 0 0" rpy="${-pi/2} 0 ${-pi/2}"/>
+    </joint>
+    <gazebo reference="sim_camera_link">
+      <sensor name="camera" type="camera">
+        <topic>camera/image</topic>
+        <camera_info_topic>camera/camera_info</camera_info_topic>
+        <update_rate>15</update_rate>
+        <gz_frame_id>sim_camera_optical_frame</gz_frame_id>
+        <always_on>1</always_on>
+        <visualize>false</visualize>
+        <camera>
+          <horizontal_fov>1.047</horizontal_fov>     <!-- ~60° HFOV -->
+          <image>
+            <!-- 320x240 to keep gz render + bridge cheap. YOLO downscales
+                 again to 192x192 for inference. Bump back to 640x480 if
+                 detection range or quality becomes the bottleneck. -->
+            <width>320</width>
+            <height>240</height>
+            <format>R8G8B8</format>
+          </image>
+          <clip>
+            <near>0.05</near>
+            <far>15.0</far>
+          </clip>
+          <noise>
+            <type>gaussian</type>
+            <mean>0.0</mean>
+            <stddev>0.007</stddev>
+          </noise>
+        </camera>
+      </sensor>
     </gazebo>
     <gazebo reference="laser_frame">
